Commit message: Fixed old refs to puck to be refs to raven

File: raven_description/urdf/d435.urdf.xacro (robot description, xacro)
@@ -8,6 +8,6 @@
 <robot name="sensor_d435" xmlns:xacro="http://ros.org/wiki/xacro">
   <!-- Includes -->
-  <xacro:include filename="$(find puck_description)/urdf/_materials.urdf.xacro" />
-  <xacro:include filename="$(find puck_description)/urdf/_usb_plug.urdf.xacro" />
+  <xacro:include filename="$(find raven_description)/urdf/_materials.urdf.xacro" />
+  <xacro:include filename="$(find raven_description)/urdf/_usb_plug.urdf.xacro" />
   <xacro:macro name="sensor_d435" params="parent *origin name:=camera use_nominal_extrinsics:=false">
     <xacro:arg name="add_plug" default="false" />
@@ -54,5 +54,5 @@
         <geometry>
           <!-- <box size="${d435_cam_width} ${d435_cam_height} ${d435_cam_depth}"/> -->
-	        <mesh filename="package://puck_description/meshes/d435.dae" />
+	        <mesh filename="package://raven_description/meshes/d435.dae" />
         </geometry>
       </visual>
