Commit message: Gazebo fixes. Sonar/LD06/TOF macros.

File: raven_description/urdf/caster.urdf.xacro (robot description, xacro)
@@ -1,5 +1,5 @@
 <?xml version="1.0"?>
 <!--
-Copyright (c) 2018 Michael Wimble
+Copyright (c) 2023 Michael Wimble
 Permission is hereby granted, free of charge, to any person obtaining a copy
 of this software and associated documentation files (the "Software"), to deal
@@ -24,5 +24,5 @@
 				<origin xyz="0 0 0" rpy="${M_PI/2} 0 0" />
 				<geometry>
-			        <cylinder length="${caster_width}" radius="${caster_radius}" />
+					<cylinder length="${caster_width}" radius="${caster_radius}" />
 				</geometry>
 			</collision>
@@ -34,7 +34,7 @@
 			<visual>
 				<geometry>
-			        <cylinder length="${caster_width}" radius="${caster_radius}" />
+					<cylinder length="${caster_width}" radius="${caster_radius}" />
 				</geometry>
-		        <material name="caster_wheel_material" />
+				<material name="caster_wheel_material" />
 				<origin xyz="0 0 0" rpy="${M_PI/2} 0 0" />
 			</visual>
@@ -45,4 +45,9 @@
 			<xacro:insert_block name="joint_pose" />
 		</joint>
+		<gazebo reference="${wheel_prefix}_wheel_link">
+			<mu1>0.00000</mu1>
+			<mu2>0.00000</mu2>
+			<material>Gazebo/Red</material>
+		</gazebo>
 	</xacro:macro>
 </robot>

File: raven_description/urdf/ld06.urdf.xacro (robot description, xacro)
@@ -51,4 +51,9 @@
       </visual>
     </link>
+    <gazebo reference="ld06_box_${lidar_prefix}">
+      <material>
+        Gazebo/Black
+      </material>
+    </gazebo>
     <link name="ld06_cylinder_${lidar_prefix}">
       <collision>
@@ -65,4 +70,9 @@
       </visual>
     </link>
+    <gazebo reference="ld06_cylinder_${lidar_prefix}">
+      <material>
+        Gazebo/BlueGlow
+      </material>
+    </gazebo>
     <link name="lidar_frame_${lidar_prefix}">
       <collision>
@@ -79,4 +89,9 @@
       </visual>
     </link>
+    <gazebo reference="ld06_frame_${lidar_prefix}">
+      <material>
+        Gazebo/Grey
+      </material>
+    </gazebo>
     <link name="ld06_base_cylinder_${lidar_prefix}">
       <collision>
@@ -93,4 +108,9 @@
       </visual>
     </link>
+    <gazebo reference="ld06_base_cylinder_${lidar_prefix}">
+      <material>
+        Gazebo/Grey
+      </material>
+    </gazebo>
     <joint name="ld06_base_cylinder_base_box_${lidar_prefix}" type="fixed">
       <parent link="lidar_frame_${lidar_prefix}" />
@@ -116,4 +136,40 @@
       <xacro:insert_block name="joint_pose" />
     </joint>
+    <gazebo reference="lidar_frame_${lidar_prefix}">
+      <sensor name="sensor_ray_${lidar_prefix}" type="ray">
+        <ray>
+          <scan>
+            <horizontal>
+              <samples>450</samples>
+              <resolution>0.8</resolution>
+              <min_angle>0</min_angle>
+              <max_angle>6.28</max_angle>
+            </horizontal>
+          </scan>
+          <range>
+            <min>0.05</min>
+            <max>10.0</max>
+          </range>
+          <noise>
+            <type>gaussian</type>
+            <mean>0.0</mean>
+            <stddev>0.02</stddev>
+          </noise>
+        </ray>
+        <always_on>true</always_on>
+        <update_rate>3.0</update_rate>
+        <plugin name="laserscan_${lidar_prefix}" filename="libgazebo_ros_ray_sensor.so">
+          <ros>
+            <remapping>~/out:=/scan_${lidar_prefix}</remapping>
+          </ros>
+          <output_type>sensor_msgs/LaserScan</output_type>
+          <frame_name>scan</frame_name>
+        </plugin>
+        <visualize>1</visualize>
+      </sensor>
+      <material>
+        Gazebo/Black
+      </material>
+    </gazebo>
   </xacro:macro>
 </robot>

File: raven_description/urdf/raven.urdf.xacro (robot description, xacro)
@@ -19,4 +19,5 @@
 -->
 <robot xmlns:xacro="http://ros.org/wiki/xacro" name="ravel">
+    <xacro:include filename="$(find raven_description)/urdf/raven_properties.urdf.xacro" />
     <xacro:include filename="$(find raven_description)/urdf/caster.urdf.xacro" />
     <xacro:include filename="$(find raven_description)/urdf/ld06.urdf.xacro" />
@@ -24,28 +25,4 @@
     <xacro:include filename="$(find raven_description)/urdf/raven_gazebo.urdf.xacro" />
     <xacro:include filename="$(find raven_description)/urdf/wheel.urdf.xacro" />
-    <material name="black">
-        <color rgba="0 0 0 1"/>
-    </material>
-    <material name="blackish">
-        <color rgba="0.1 0.1 0.1 1"/>
-    </material>
-    <xacro:property name="M_PI" value="3.14159" />
-    <xacro:property name="body_height" value="0.262" />
-    <xacro:property name="body_length" value="0.4572" />
-    <xacro:property name="body_width" value="0.3048" />
-    <xacro:property name="caster_radius" value="0.0381" />
-    <xacro:property name="caster_width" value="0.023" />
-    <xacro:property name="fwheel_offset" value="0.170" />
-    <xacro:property name="gear_box_center_height" value="0.015" />
-    <xacro:property name="t265_height" value="0.016" />
-    <xacro:property name="t265_length" value="0.100" />
-    <xacro:property name="t265_width" value="0.008" />
-    <xacro:property name="t265_x_offset" value="0.2126" />
-    <xacro:property name="wheel_radius" value="0.10" />
-    <xacro:property name="wheel_center_offset" value="0.030" />
-    <xacro:property name="wheel_width" value="0.0254" />
-    <xacro:property name="base_to_floor_z_offset" value="${wheel_radius+gear_box_center_height}" />
-    <xacro:property name="t265_z_offset" value="${base_to_floor_z_offset+0.293}" />
-    <xacro:property name="wheel_offset_from_front" value="${body_length/2}" />
     <link name="base_link">
         <collision>
@@ -60,19 +37,35 @@
             </geometry>
             <material name="aluminum_frame" />
-            <origin rpy="0 0 0" xyz="${(-body_length/2)+wheel_offset_from_front} 0 ${(body_height/2)}" />
+            <origin rpy="0 0 0"
+                xyz="${(-body_length/2)+wheel_offset_from_front} 0 ${(body_height/2)}" />
         </visual>
+        <inertial>
+            <origin xyz="0 0 0.05" rpy="0 0 0" />
+            <mass value="12" />
+            <inertia
+                ixx="${(1/12) * mass * ((body_width  * body_width)  + (body_height * body_height))}"
+                ixy="0.0" ixz="0.0"
+                iyy="${(1/12) * mass * ((body_length * body_length) + (body_height * body_height))}"
+                iyz="0.0"
+                izz="${(1/12) * mass * ((body_length * body_length) + (body_width  * body_width))}" />
+        </inertial>
     </link>
+    <gazebo
+        reference="base_link">
+        <material>
+            aluminum_frame
+        </material>
+    </gazebo>
     <link name="base_footprint" />
     <link name="odom" />
     <link name="odom_frame" />
     <joint name="odom_to_odom_frame_joint" type="fixed">
-        <origin xyz="0 0 0" rpy="0 0 0" />>
-        <parent link="odom" />
+        <origin xyz="0 0 0" rpy="0 0 0" />> <parent link="odom" />
         <child link="odom_frame" />
     </joint>
     <joint name="odom_frame_to_t265_pose_frame_joint" type="fixed">
-        <origin xyz="0 0 0" rpy="0 0 0" />>
-        <parent link="odom_frame" />
-        <child link="t265_pose_frame" />
+        <origin xyz="0 0 0" rpy="0 0 0" />> <parent link="odom_frame" />
+        <child
+            link="t265_pose_frame" />
     </joint>
     <joint name="base_footprint_joint" type="fixed">
@@ -85,17 +78,22 @@
     </xacro:wheel>
     <xacro:wheel wheel_prefix="front_right">
-        <origin xyz="0 -${(body_width/2)+wheel_center_offset} -${gear_box_center_height}" rpy="0 0 0" />
+        <origin xyz="0 -${(body_width/2)+wheel_center_offset} -${gear_box_center_height}"
+            rpy="0 0 0" />
     </xacro:wheel>
     <xacro:caster wheel_prefix="fcaster">
-        <origin xyz="${fwheel_offset} 0.0 -${wheel_radius + gear_box_center_height - caster_radius}" rpy="0 0 0" />
+        <origin xyz="${fwheel_offset} 0.0 -${wheel_radius + gear_box_center_height - caster_radius}"
+            rpy="0 0 0" />
     </xacro:caster>
     <xacro:caster wheel_prefix="rcaster">
-        <origin xyz="${-fwheel_offset} 0.0 -${wheel_radius + gear_box_center_height - caster_radius}" rpy="0 0 0" />
+        <origin
+            xyz="${-fwheel_offset} 0.0 -${wheel_radius + gear_box_center_height - caster_radius}"
+            rpy="0 0 0" />
     </xacro:caster>
     <xacro:ld06 lidar_prefix="right_rear">
-        <origin xyz="${-(body_length / 2) - 0.030}  -${((body_width / 2) - 0)} 0.200" rpy="0 0 ${M_PI}"/>
+        <origin xyz="${-(body_length / 2) - 0.030}  -${((body_width / 2) - 0)} 0.200"
+            rpy="0 0 ${M_PI}" />
     </xacro:ld06>
     <xacro:ld06 lidar_prefix="left_front">
-        <origin xyz="${(body_length / 2) + 0.030}  ${((body_width / 2) - 0.0)} 0.040" rpy="0 0 0"/>
+        <origin xyz="${(body_length / 2) + 0.030}  ${((body_width / 2) - 0.0)} 0.040" rpy="0 0 0" />
     </xacro:ld06>
     <!-- T265 y tilt is 31 degrees or 0.541 radians -->
@@ -116,9 +114,14 @@
         </visual>
     </link>
+    <gazebo reference="t265_pose_frame">
+        <material>
+            Gazebo/DarkGrey
+        </material>
+    </gazebo>
     <joint name="t265_to_base_footprint" type="fixed">
         <parent link="t265_rotate_frame" />
         <child link="base_footprint" />
         <origin xyz="-${t265_x_offset} 0 -${t265_z_offset}" rpy="0 0 0" />
-         <!--
+        <!--
         <child link="base_footprint" />
         <origin xyz="-${t265_x_offset} 0 -${t265_z_offset}" rpy="0 0.541 0 " />

File: raven_description/urdf/raven_gazebo.urdf.xacro (robot description, xacro)
@@ -120,234 +120,11 @@
     <child link="odom" />
   </joint> -->
-  <gazebo reference="base_link">
-    <material>
-      aluminum_frame
-    </material>
-    <inertial>
-      <origin xyz="0 0 0.05" rpy="0 0 0" />
-      <mass value="12" />
-      <inertia ixx="2.26" ixy="0.0" ixz="0.0" iyy="6.26" iyz="0.0" izz="8.5" />
-    </inertial>
-  </gazebo>
-  <gazebo reference="ld06_base_cylinder_left_front">
-    <material>
-      Gazebo/Grey
-    </material>
-  </gazebo>
-  <gazebo reference="ld06_base_cylinder_right_rear">
-    <material>
-      Gazebo/Grey
-    </material>
-  </gazebo>
-  <gazebo reference="ld06_box_left_front">
-    <material>
-      Gazebo/Black
-    </material>
-  </gazebo>
-  <gazebo reference="ld06_box_right_rear">
-    <material>
-      Gazebo/Black
-    </material>
-  </gazebo>
-  <gazebo reference="ld06_cylinder_left_front">
-    <material>
-      Gazebo/BlueGlow
-    </material>
-  </gazebo>
-  <gazebo reference="ld06_cylinder_right_rear">
-    <material>
-      Gazebo/BlueGlow
-    </material>
-  </gazebo>
-  <gazebo reference="ld06_frame_left_front">
-    <material>
-      Gazebo/Grey
-    </material>
-  </gazebo>
-  <gazebo reference="ld06_frame_right_rear">
-    <material>
-      Gazebo/Grey
-    </material>
-  </gazebo>
-  <gazebo reference="sonar_0">
-    <material>
-      Gazebo/Black
-    </material>
-  </gazebo>
-  <gazebo reference="sonar_1">
-    <material>
-      Gazebo/Black
-    </material>
-  </gazebo>
-  <gazebo reference="sonar_2">
-    <material>
-      Gazebo/Black
-    </material>
-  </gazebo>
-  <gazebo reference="sonar_3">
-    <material>
-      Gazebo/Black
-    </material>
-  </gazebo>
-  <gazebo reference="tof_0">
-    <material>
-      Gazebo/Grey
-    </material>
-  </gazebo>
-  <gazebo reference="tof_1">
-    <material>
-      Gazebo/Grey
-    </material>
-  </gazebo>
-  <gazebo reference="tof_2">
-    <material>
-      Gazebo/Grey
-    </material>
-  </gazebo>
-  <gazebo reference="tof_3">
-    <material>
-      Gazebo/Grey
-    </material>
-  </gazebo>
-  <gazebo reference="tof_4">
-    <material>
-      Gazebo/Grey
-    </material>
-  </gazebo>
-  <gazebo reference="tof_5">
-    <material>
-      Gazebo/Grey
-    </material>
-  </gazebo>
-  <gazebo reference="tof_6">
-    <material>
-      Gazebo/Grey
-    </material>
-  </gazebo>
-  <gazebo reference="tof_7">
-    <material>
-      Gazebo/Grey
-    </material>
-  </gazebo>
-  <gazebo reference="t265_pose_frame">
-    <material>
-      Gazebo/DarkGrey
-    </material>
-  </gazebo>
-  <gazebo reference="lidar_frame_right_rear">
-    <sensor name="sensor_ray_right" type="ray">
-      <ray>
-        <scan>
-          <horizontal>
-            <samples>450</samples>
-            <resolution>0.8</resolution>
-            <min_angle>0</min_angle>
-            <max_angle>6.28</max_angle>
-          </horizontal>
-        </scan>
-        <range>
-          <min>0.05</min>
-          <max>10.0</max>
-        </range>
-        <noise>
-          <type>gaussian</type>
-          <mean>0.0</mean>
-          <stddev>0.02</stddev>
-        </noise>
-      </ray>
-      <always_on>true</always_on>
-      <update_rate>3.0</update_rate>
-      <plugin name="laserscan_right" filename="libgazebo_ros_ray_sensor.so">
-        <ros>
-          <remapping>~/out:=/scan_right</remapping>
-        </ros>
-        <output_type>sensor_msgs/LaserScan</output_type>
-        <frame_name>scan</frame_name>
-      </plugin>
-      <visualize>1</visualize>
-    </sensor>
-    <material>
-      Gazebo/Black
-    </material>
-  </gazebo>
-  <gazebo reference="lidar_frame_left_front">
-    <sensor name="sensor_ray_left" type="ray">
-      <ray>
-        <scan>
-          <horizontal>
-            <samples>450</samples>
-            <resolution>0.8</resolution>
-            <min_angle>0</min_angle>
-            <max_angle>6.28</max_angle>
-          </horizontal>
-        </scan>
-        <range>
-          <min>0.05</min>
-          <max>10.0</max>
-        </range>
-        <noise>
-          <type>gaussian</type>
-          <mean>0.0</mean>
-          <stddev>0.02</stddev>
-        </noise>
-      </ray>
-      <always_on>true</always_on>
-      <update_rate>3.0</update_rate>
-      <plugin name="laserscan_left" filename="libgazebo_ros_ray_sensor.so">
-        <ros>
-          <remapping>~/out:=/scan_right</remapping>
-        </ros>
-        <output_type>sensor_msgs/LaserScan</output_type>
-        <frame_name>scan</frame_name>
-      </plugin>
-      <visualize>1</visualize>
-    </sensor>
-    <material>
-      Gazebo/Black
-    </material>
-  </gazebo>
-  <gazebo reference="front_left_wheel_link">
-    <mu1>200.0</mu1>
-    <mu2>100.0</mu2>
-    <kp>1000000.0</kp>
-    <kd>1.0</kd>
-    <max_vel>0.01</max_vel>
-    <min_depth>0.001</min_depth>
-    <material>Gazebo/Black</material>
-  </gazebo>
-  <gazebo reference="front_right_wheel_link">
-    <mu1>200.0</mu1>
-    <mu2>100.0</mu2>
-    <kp>1000000.0</kp>
-    <kd>1.0</kd>
-    <max_vel>0.01</max_vel>
-    <min_depth>0.001</min_depth>
-    <material>Gazebo/Black</material>
-  </gazebo>
-  <gazebo reference="fcaster_wheel_link">
-    <mu1>0.00000</mu1>
-    <mu2>0.00000</mu2>
-    <!-- kp>100000.0</kp>
-    <kd>1.0</kd  -->
-    <max_vel>0.001</max_vel>
-    <min_depth>0.0001</min_depth>
-    <material>Gazebo/Red</material>
-  </gazebo>
-  <gazebo reference="rcaster_wheel_link">
-    <mu1>0.00000</mu1>
-    <mu2>0.00000</mu2>
-    <!-- kp>100000.0</kp>
-    <kd>1.0</kd  -->
-    <max_vel>0.001</max_vel>
-    <min_depth>0.0001</min_depth>
-    <material>Gazebo/Red</material>
-  </gazebo>
   <gazebo>
     <plugin name='diff_drive_simbot' filename='libgazebo_ros_diff_drive.so'>
-      <ros>
+      <!-- <ros>
         <namespace>/simbot</namespace>
         <remapping>cmd_vel:=/cmd_vel</remapping>
         <remapping>odom:=/odom</remapping>
-      </ros>
+      </ros> -->
       <!-- wheels -->
       <left_joint>front_left_wheel</left_joint>
@@ -356,5 +133,5 @@
       <wheel_separation>0.3108</wheel_separation>
       <wheel_diameter>0.2</wheel_diameter>
-      <update_rate>100.0</update_rate>
+      <update_rate>80.0</update_rate>
       <!-- limits -->
       <max_wheel_torque>8.0</max_wheel_torque>
@@ -365,5 +142,5 @@
       <publish_wheel_tf>true</publish_wheel_tf>
       <odometry_frame>odom_frame</odometry_frame>
-      <robot_base_frame>base_footprint</robot_base_frame>
+      <robot_base_frame>base_link</robot_base_frame>
     </plugin>
     <plugin name="gazebo_ros_joint_state_publisher"
@@ -376,5 +153,5 @@
       </ros>
       <!-- Update rate in Hertz -->
-      <update_rate>500</update_rate>
+      <update_rate>80</update_rate>
       <!-- Name of joints in the model whose states will be published. -->
       <joint_name>front_left_wheel</joint_name>

File: raven_description/urdf/sonar.urdf.xacro (robot description, xacro)
@@ -27,59 +27,39 @@
     <xacro:property name="sonar_width" value="0.050" />
     <xacro:property name="sonar_z_offset" value="0.173" />
-    <link name="sonar_0">
-        <visual>
-            <geometry>
-                <box size="${sonar_depth} ${sonar_width} ${sonar_height}" />
-            </geometry>
-            <material name="black" />
-            <origin xyz="0 0 0" rpy="0 0 0" />
-        </visual>
-    </link>
-    <joint name="baselink_to_sonar_0" type="fixed">
-        <child link="sonar_0" />
-        <parent link="base_link" />
+    <xacro:macro name="sonar_unit" params="number *joint_pose">
+        <link name="sonar_${number}">
+            <visual>
+                <geometry>
+                    <box size="${sonar_depth} ${sonar_width} ${sonar_height}" />
+                </geometry>
+                <material name="black" />
+                <origin xyz="0 0 0" rpy="0 0 0" />
+            </visual>
+        </link>
+        <joint name="baselink_to_sonar_${number}" type="fixed">
+            <child link="sonar_${number}" />
+            <parent link="base_link" />
+            <xacro:insert_block name="joint_pose" />
+        </joint>
+        <gazebo reference="sonar_${number}">
+            <material>
+                Gazebo/Black
+            </material>
+        </gazebo>
+    </xacro:macro>
+    <xacro:sonar_unit number="0">
         <origin xyz="${front_edge+(sonar_depth/2)} 0 ${(sonar_height/2)+sonar_z_offset}" rpy="0 0 0" />
-    </joint>
-    <link name="sonar_1">
-        <visual>
-            <geometry>
-                <box size="${sonar_depth} ${sonar_width} ${sonar_height}" />
-            </geometry>
-            <material name="black" />
-            <origin xyz="0 0 0" rpy="0 0 0" />
-        </visual>
-    </link>
-    <joint name="baselink_to_sonar_1" type="fixed">
-        <child link="sonar_1" />
-        <parent link="base_link" />
-        <origin xyz="0 ${case_left_edge+(sonar_depth/2)} ${(sonar_height/2)+sonar_z_offset}" rpy="0 0 ${M_PI / 2}" />
-    </joint>
-    <link name="sonar_2">
-        <visual>
-            <geometry>
-                <box size="${sonar_depth} ${sonar_width} ${sonar_height}" />
-            </geometry>
-            <material name="black" />
-            <origin xyz="0 0 0" rpy="0 0 0" />
-        </visual>
-    </link>
-    <joint name="baselink_to_sonar_2" type="fixed">
-        <child link="sonar_2" />
-        <parent link="base_link" />
-        <origin xyz="0 ${case_right_edge-(sonar_depth/2)} ${(sonar_height/2)+sonar_z_offset}" rpy="0 0 -${M_PI / 2}" />
-    </joint>
-    <link name="sonar_3">
-        <visual>
-            <geometry>
-                <box size="${sonar_depth} ${sonar_width} ${sonar_height}" />
-            </geometry>
-            <material name="black" />
-            <origin xyz="0 0 0" rpy="0 0 0" />
-        </visual>
-    </link>
-    <joint name="baselink_to_sonar_3" type="fixed">
-        <child link="sonar_3" />
-        <parent link="base_link" />
-        <origin xyz="${back_edge-(sonar_depth/2)} 0 ${(sonar_height/2)+sonar_z_offset}" rpy="0 0 ${M_PI}" />
-    </joint>
+    </xacro:sonar_unit>
+    <xacro:sonar_unit number="1">
+        <origin xyz="0 ${case_left_edge+(sonar_depth/2)} ${(sonar_height/2)+sonar_z_offset}"
+            rpy="0 0 ${M_PI / 2}" />
+    </xacro:sonar_unit>
+    <xacro:sonar_unit number="2">
+        <origin xyz="0 ${case_right_edge-(sonar_depth/2)} ${(sonar_height/2)+sonar_z_offset}"
+            rpy="0 0 -${M_PI / 2}" />
+    </xacro:sonar_unit>
+    <xacro:sonar_unit number="3">
+        <origin xyz="${back_edge-(sonar_depth/2)} 0 ${(sonar_height/2)+sonar_z_offset}"
+            rpy="0 0 ${M_PI}" />
+    </xacro:sonar_unit>
 </robot>
