Commit message: Gazebo fixes. Sonar/LD06/TOF macros.

File: raven_description/urdf/time_of_flight.urdf.xacro (robot description, xacro)
@@ -27,115 +27,64 @@
     <xacro:property name="tof_width" value="0.023" />
     <xacro:property name="tof_z_offset" value="0.015" />
-    <link name="tof_0">
-        <visual>
-            <geometry>
-                <box size="${tof_depth} ${tof_width} ${tof_height}" />
-            </geometry>
-            <material name="black" />
-            <origin xyz="0 0 0" rpy="0 0 0" />
-        </visual>
-    </link>
-    <joint name="baselink_to_tof_0" type="fixed">
-        <child link="tof_0" />
-        <parent link="base_link" />
-        <origin xyz="${front_edge+(tof_depth/2)} ${case_left_edge-(tof_width/2) - 0.020} ${(tof_height/2)+tof_z_offset}" rpy="0 0 0" />
-    </joint>
-    <link name="tof_1">
-        <visual>
-            <geometry>
-                <box size="${tof_depth} ${tof_width} ${tof_height}" />
-            </geometry>
-            <material name="black" />
-            <origin xyz="0 0 0" rpy="0 0 0" />
-        </visual>
-    </link>
-    <joint name="baselink_to_tof_1" type="fixed">
-        <child link="tof_1" />
-        <parent link="base_link" />
-        <origin xyz="${front_edge+(tof_depth/2)} ${case_right_edge +(tof_width/2) + 0.020} ${(tof_height/2)+tof_z_offset}" rpy="0 0 0" />
-    </joint>
-    <link name="tof_2">
-        <visual>
-            <geometry>
-                <box size="${tof_depth} ${tof_width} ${tof_height}" />
-            </geometry>
-            <material name="black" />
-            <origin xyz="0 0 0" rpy="0 0 0" />
-        </visual>
-    </link>
-    <joint name="baselink_to_tof_2" type="fixed">
-        <child link="tof_2" />
-        <parent link="base_link" />
-        <origin xyz="${front_edge-(tof_width/2 + 0.020)} ${case_left_edge+(tof_depth/2)} ${(tof_height/2)+tof_z_offset}" rpy="0 0 ${M_PI / 2}" />
-    </joint>
-    <link name="tof_3">
-        <visual>
-            <geometry>
-                <box size="${tof_depth} ${tof_width} ${tof_height}" />
-            </geometry>
-            <material name="black" />
-            <origin xyz="0 0 0" rpy="0 0 0" />
-        </visual>
-    </link>
-    <joint name="baselink_to_tof_3" type="fixed">
-        <child link="tof_3" />
-        <parent link="base_link" />
-        <origin xyz="${front_edge-(tof_width/2 + 0.020)} ${case_right_edge-(tof_depth/2)} ${(tof_height/2)+tof_z_offset}" rpy="0 0 -${M_PI / 2}" />
-    </joint>
-    <link name="tof_4">
-        <visual>
-            <geometry>
-                <box size="${tof_depth} ${tof_width} ${tof_height}" />
-            </geometry>
-            <material name="black" />
-            <origin xyz="0 0 0" rpy="0 0 0" />
-        </visual>
-    </link>
-    <joint name="baselink_to_tof_4" type="fixed">
-        <child link="tof_4" />
-        <parent link="base_link" />
-        <origin xyz="${back_edge+(tof_width/2) + 0.020} ${case_left_edge+(tof_depth/2)} ${(tof_height/2)+tof_z_offset}" rpy="0 0 ${M_PI / 2}" />
-    </joint>
-    <link name="tof_5">
-        <visual>
-            <geometry>
-                <box size="${tof_depth} ${tof_width} ${tof_height}" />
-            </geometry>
-            <material name="black" />
-            <origin xyz="0 0 0" rpy="0 0 0" />
-        </visual>
-    </link>
-    <joint name="baselink_to_tof_5" type="fixed">
-        <child link="tof_5" />
-        <parent link="base_link" />
-        <origin xyz="${back_edge+(tof_width/2) + 0.020} ${case_right_edge-(tof_depth/2)} ${(tof_height/2)+tof_z_offset}" rpy="0 0 -${M_PI / 2}" />
-    </joint>
-    <link name="tof_6">
-        <visual>
-            <geometry>
-                <box size="${tof_depth} ${tof_width} ${tof_height}" />
-            </geometry>
-            <material name="black" />
-            <origin xyz="0 0 0" rpy="0 0 0" />
-        </visual>
-    </link>
-    <joint name="baselink_to_tof_6" type="fixed">
-        <child link="tof_6" />
-        <parent link="base_link" />
-        <origin xyz="${back_edge-(tof_depth/2)} ${case_left_edge-(tof_width/2) - 0.020} ${(tof_height/2)+tof_z_offset}" rpy="0 0 -${M_PI}" />
-    </joint>
-    <link name="tof_7">
-        <visual>
-            <geometry>
-                <box size="${tof_depth} ${tof_width} ${tof_height}" />
-            </geometry>
-            <material name="black" />
-            <origin xyz="0 0 0" rpy="0 0 0" />
-        </visual>
-    </link>
-    <joint name="baselink_to_tof_7" type="fixed">
-        <child link="tof_7" />
-        <parent link="base_link" />
-        <origin xyz="${back_edge-(tof_depth/2)} ${case_right_edge+(tof_width/2) + 0.020} ${(tof_height/2)+tof_z_offset}" rpy="0 0 -${M_PI}" />
-    </joint>
+    <xacro:macro name="tof_unit" params="number *joint_pose">
+        <link name="tof_${number}">
+            <visual>
+                <geometry>
+                    <box size="${tof_depth} ${tof_width} ${tof_height}" />
+                </geometry>
+                <material name="black" />
+                <origin xyz="0 0 0" rpy="0 0 0" />
+            </visual>
+        </link>
+        <joint name="baselink_to_tof_${number}" type="fixed">
+            <child link="tof_${number}" />
+            <parent link="base_link" />
+            <xacro:insert_block name="joint_pose" />
+        </joint>
+        <gazebo reference="tof_${number}">
+            <material>
+                Gazebo/Grey
+            </material>
+        </gazebo>
+    </xacro:macro>
+    <xacro:tof_unit number="0">
+        <origin
+            xyz="${front_edge+(tof_depth/2)} ${case_left_edge-(tof_width/2) - 0.020} ${(tof_height/2)+tof_z_offset}"
+            rpy="0 0 0" />
+    </xacro:tof_unit>
+    <xacro:tof_unit number="1">
+        <origin
+            xyz="${front_edge+(tof_depth/2)} ${case_right_edge +(tof_width/2) + 0.020} ${(tof_height/2)+tof_z_offset}"
+            rpy="0 0 0" />
+    </xacro:tof_unit>
+    <xacro:tof_unit number="2">
+        <origin
+            xyz="${front_edge-(tof_width/2 + 0.020)} ${case_left_edge+(tof_depth/2)} ${(tof_height/2)+tof_z_offset}"
+            rpy="0 0 ${M_PI / 2}" />
+    </xacro:tof_unit>
+    <xacro:tof_unit number="3">
+        <origin
+            xyz="${front_edge-(tof_width/2 + 0.020)} ${case_right_edge-(tof_depth/2)} ${(tof_height/2)+tof_z_offset}"
+            rpy="0 0 -${M_PI / 2}" />
+    </xacro:tof_unit>
+    <xacro:tof_unit number="4">
+        <origin
+            xyz="${back_edge+(tof_width/2) + 0.020} ${case_left_edge+(tof_depth/2)} ${(tof_height/2)+tof_z_offset}"
+            rpy="0 0 ${M_PI / 2}" />
+    </xacro:tof_unit>
+    <xacro:tof_unit number="5">
+        <origin
+            xyz="${back_edge+(tof_width/2) + 0.020} ${case_right_edge-(tof_depth/2)} ${(tof_height/2)+tof_z_offset}"
+            rpy="0 0 -${M_PI / 2}" />
+    </xacro:tof_unit>
+    <xacro:tof_unit number="6">
+        <origin
+            xyz="${back_edge-(tof_depth/2)} ${case_left_edge-(tof_width/2) - 0.020} ${(tof_height/2)+tof_z_offset}"
+            rpy="0 0 -${M_PI}" />
+    </xacro:tof_unit>
+    <xacro:tof_unit number="7">
+        <origin
+            xyz="${back_edge-(tof_depth/2)} ${case_right_edge+(tof_width/2) + 0.020} ${(tof_height/2)+tof_z_offset}"
+            rpy="0 0 -${M_PI}" />
+    </xacro:tof_unit>
 </robot>

File: raven_description/urdf/wheel.urdf.xacro (robot description, xacro)
@@ -1,5 +1,5 @@
 <?xml version="1.0"?>
 <!--
-Copyright (c) 2018 Michael Wimble
+Copyright (c) 2023 Michael Wimble
 Permission is hereby granted, free of charge, to any person obtaining a copy
 of this software and associated documentation files (the "Software"), to deal
@@ -24,5 +24,5 @@
 				<origin xyz="0 0 0" rpy="${M_PI/2} 0 0" />
 				<geometry>
-			        <cylinder length="${wheel_width}" radius="${wheel_radius}" />
+					<cylinder length="${wheel_width}" radius="${wheel_radius}" />
 				</geometry>
 			</collision>
@@ -30,10 +30,10 @@
 				<mass value="2.637" />
 				<origin xyz="0 0 0" />
-				<inertia  ixx="0.02467" ixy="0" ixz="0" iyy="0.04411" iyz="0" izz="0.02467" />
+				<inertia ixx="0.02467" ixy="0" ixz="0" iyy="0.04411" iyz="0" izz="0.02467" />
 			</inertial>
 			<visual>
 				<origin xyz="0 0 0" rpy="${M_PI/2} 0 0" />
 				<geometry>
-			        <cylinder length="${wheel_width}" radius="${wheel_radius}" />
+					<cylinder length="${wheel_width}" radius="${wheel_radius}" />
 				</geometry>
 				<material name="wheel_material" />
@@ -41,10 +41,10 @@
 		</link>
 		<joint name="${wheel_prefix}_wheel" type="continuous">
-			<parent link="base_link"/>
-			<child link="${wheel_prefix}_wheel_link"/>
-			<xacro:insert_block name="joint_pose"/>
+			<parent link="base_link" />
+			<child link="${wheel_prefix}_wheel_link" />
+			<xacro:insert_block name="joint_pose" />
 			<axis xyz="0 1 0" rpy="0 0 0" />
-		    <limit effort="100" velocity="100"/>
-		    <joint_properties damping="0.1" friction="0.5"/>
+			<limit effort="100" velocity="3" />
+			<dynamics damping="0.1" friction="0.5" />
 		</joint>
 		<transmission name="${wheel_prefix}_wheel_trans" type="SimpleTransmission">
@@ -57,4 +57,17 @@
 			</joint>
 		</transmission>
+		<gazebo reference="${wheel_prefix}_wheel_link">
+			<mu1 value="10000.0" />
+			<mu2 value="10000.0" />
+			<kp value="1e13" />
+			<kd value="1" />
+			<!-- <mu1>200.0</mu1>
+			<mu2>100.0</mu2>
+			<kp>1000000.0</kp>
+			<kd>1.0</kd>
+			<max_vel>0.01</max_vel>
+			<min_depth>0.001</min_depth> -->
+			<material>Gazebo/Black</material>
+		</gazebo>
 	</xacro:macro>
 </robot>

Commit message: Partial frame fixes for gazebo

File: raven_description/urdf/caster.urdf.xacro (robot description, xacro)
@@ -40,5 +40,5 @@
 			</visual>
 		</link>
-		<joint name="${wheel_prefix}_wheel" type="fixed">
+		<joint name="${wheel_prefix}_wheel" type="continuous">
 			<parent link="base_link" />
 			<child link="${wheel_prefix}_wheel_link" />

File: raven_description/urdf/ld06.urdf.xacro (robot description, xacro)
@@ -158,5 +158,5 @@
         </ray>
         <always_on>true</always_on>
-        <update_rate>3.0</update_rate>
+        <update_rate>10.0</update_rate>
         <plugin name="laserscan_${lidar_prefix}" filename="libgazebo_ros_ray_sensor.so">
           <ros>
@@ -164,5 +164,5 @@
           </ros>
           <output_type>sensor_msgs/LaserScan</output_type>
-          <frame_name>scan</frame_name>
+          <frame_name>lidar_frame_${lidar_prefix}</frame_name>
         </plugin>
         <visualize>1</visualize>

File: raven_description/urdf/wheel.urdf.xacro (robot description, xacro)
@@ -48,13 +48,4 @@
 			<dynamics damping="0.1" friction="0.5" />
 		</joint>
-		<transmission name="${wheel_prefix}_wheel_trans" type="SimpleTransmission">
-			<type>transmission_interface/SimpleTransmission</type>
-			<actuator name="${wheel_prefix}_wheel_motor">
-				<mechanicalReduction>1</mechanicalReduction>
-			</actuator>
-			<joint name="${wheel_prefix}_wheel">
-				<hardwareInterface>hardware_interface/VelocityJointInterface</hardwareInterface>
-			</joint>
-		</transmission>
 		<gazebo reference="${wheel_prefix}_wheel_link">
 			<mu1 value="10000.0" />

Commit message: Simulator seems to be working with 2 OAK-D cameras

File: raven_description/urdf/caster.urdf.xacro (robot description, xacro)
@@ -40,5 +40,5 @@
 			</visual>
 		</link>
-		<joint name="${wheel_prefix}_wheel" type="continuous">
+		<joint name="${wheel_prefix}_wheel" type="fixed">
 			<parent link="base_link" />
 			<child link="${wheel_prefix}_wheel_link" />
@@ -46,6 +46,6 @@
 		</joint>
 		<gazebo reference="${wheel_prefix}_wheel_link">
-			<mu1>0.00000</mu1>
-			<mu2>0.00000</mu2>
+			<mu1>0.00001</mu1>
+			<mu2>0.00001</mu2>
 			<material>Gazebo/Red</material>
 		</gazebo>

File: raven_description/urdf/raven_wot265.urdf.xacro (robot description, xacro)
@@ -19,4 +19,5 @@
 -->
 <robot xmlns:xacro="http://ros.org/wiki/xacro" name="ravel">
+    <xacro:include filename="$(find raven_description)/urdf/inertials.xacro" />
     <xacro:include filename="$(find raven_description)/urdf/raven_properties.urdf.xacro" />
     <xacro:include filename="$(find raven_description)/urdf/caster.urdf.xacro" />
@@ -25,4 +26,5 @@
     <xacro:include filename="$(find raven_description)/urdf/raven_gazebo.urdf.xacro" />
     <xacro:include filename="$(find raven_description)/urdf/wheel.urdf.xacro" />
+    <xacro:include filename="$(find raven_description)/urdf/oakd.urdf.xacro" />
     <link name="base_link">
         <collision>
@@ -88,3 +90,11 @@
     <xacro:include filename="$(find raven_description)/urdf/time_of_flight.urdf.xacro" />
     <xacro:include filename="$(find raven_description)/urdf/sonar.urdf.xacro" />
+    <xacro:oakd_link mount_point="right" />
+    <xacro:oakd_joint mount_point="right">
+        <origin xyz="0.170 -0.055 0.350" rpy="0 0 -0.523599" />
+    </xacro:oakd_joint>
+    <xacro:oakd_link mount_point="left" />
+    <xacro:oakd_joint mount_point="left">
+        <origin xyz="0.170 0.055 0.350" rpy="0 0 0.523599" />
+    </xacro:oakd_joint>
 </robot>
