Commit message: New URDF w/o t265 for sim. New wheel joint names.

File: raven_description/urdf/raven_gazebo.urdf.xacro (robot description, xacro)
@@ -128,13 +128,13 @@
       </ros> -->
       <!-- wheels -->
-      <left_joint>front_left_wheel</left_joint>
-      <right_joint>front_right_wheel</right_joint>
+      <left_joint>front_left_wheel_joint</left_joint>
+      <right_joint>front_right_wheel_joint</right_joint>
       <!-- kinematics -->
-      <wheel_separation>0.3108</wheel_separation>
-      <wheel_diameter>0.2</wheel_diameter>
+      <wheel_separation>${body_width * (2 * wheel_center_offset)}</wheel_separation>
+      <wheel_diameter>${wheel_radius * 2}</wheel_diameter>
       <update_rate>80.0</update_rate>
       <!-- limits -->
       <max_wheel_torque>8.0</max_wheel_torque>
-      <max_wheel_acceleration>1.0</max_wheel_acceleration>
+      <max_wheel_acceleration>1.5</max_wheel_acceleration>
       <!-- output -->
       <publish_odom>true</publish_odom>
@@ -142,5 +142,5 @@
       <publish_wheel_tf>true</publish_wheel_tf>
       <odometry_frame>odom_frame</odometry_frame>
-      <robot_base_frame>base_link</robot_base_frame>
+      <robot_base_frame>base_footprint</robot_base_frame>
     </plugin>
     <plugin name="gazebo_ros_joint_state_publisher"
@@ -155,6 +155,6 @@
       <update_rate>80</update_rate>
       <!-- Name of joints in the model whose states will be published. -->
-      <joint_name>front_left_wheel</joint_name>
-      <joint_name>front_right_wheel</joint_name>
+      <joint_name>front_left_wheel_joint</joint_name>
+      <joint_name>front_right_wheel_joint</joint_name>
     </plugin>
   </gazebo>

File: raven_description/urdf/wheel.urdf.xacro (robot description, xacro)
@@ -40,5 +40,5 @@
 			</visual>
 		</link>
-		<joint name="${wheel_prefix}_wheel" type="continuous">
+		<joint name="${wheel_prefix}_wheel_joint" type="continuous">
 			<parent link="base_link" />
 			<child link="${wheel_prefix}_wheel_link" />

Commit message: snapshot for sim

File: raven_description/urdf/raven_gazebo.urdf.xacro (robot description, xacro)
@@ -121,10 +121,8 @@
   </joint> -->
   <gazebo>
-    <plugin name='diff_drive_raven' filename='libgazebo_ros_diff_drive.so'>
-      <!-- <ros>
-        <namespace>/simbot</namespace>
-        <remapping>cmd_vel:=/cmd_vel</remapping>
-        <remapping>odom:=/odom</remapping>
-      </ros> -->
+    <plugin name='diff_drive_controller' filename='libgazebo_ros_diff_drive.so'>
+      <ros>
+        <argument>odom:=/odom</argument>
+      </ros>
       <!-- wheels -->
       <left_joint>front_left_wheel_joint</left_joint>
@@ -141,20 +139,6 @@
       <publish_odom_tf>true</publish_odom_tf>
       <publish_wheel_tf>true</publish_wheel_tf>
-      <odometry_frame>odom_frame</odometry_frame>
+      <odometry_frame>odom</odometry_frame>
       <robot_base_frame>base_footprint</robot_base_frame>
-    </plugin>
-    <plugin name="gazebo_ros_joint_state_publisher"
-      filename="libgazebo_ros_joint_state_publisher.so">
-      <ros>
-        <!-- Add a namespace -->
-        <namespace>/simbot</namespace>
-        <!-- Remap the default topic -->
-        <remapping>joint_states:=/base_wheel_joints</remapping>
-      </ros>
-      <!-- Update rate in Hertz -->
-      <update_rate>80</update_rate>
-      <!-- Name of joints in the model whose states will be published. -->
-      <joint_name>front_left_wheel_joint</joint_name>
-      <joint_name>front_right_wheel_joint</joint_name>
     </plugin>
   </gazebo>

File: raven_description/urdf/raven_wot265.urdf.xacro (robot description, xacro)
@@ -39,20 +39,13 @@
             </geometry>
             <material name="aluminum_frame" />
-            <origin rpy="0 0 0"
-                xyz="${(-body_length/2)+wheel_offset_from_front} 0 ${(body_height/2)}" />
+            <origin rpy="0 0 0" xyz="${(-body_length/2)+wheel_offset_from_front} 0 ${(body_height/2)}" />
         </visual>
         <inertial>
             <origin xyz="0 0 0.05" rpy="0 0 0" />
             <mass value="12" />
-            <inertia
-                ixx="${(1/12) * mass * ((body_width  * body_width)  + (body_height * body_height))}"
-                ixy="0.0" ixz="0.0"
-                iyy="${(1/12) * mass * ((body_length * body_length) + (body_height * body_height))}"
-                iyz="0.0"
-                izz="${(1/12) * mass * ((body_length * body_length) + (body_width  * body_width))}" />
+            <inertia ixx="${(1/12) * mass * ((body_width  * body_width)  + (body_height * body_height))}" ixy="0.0" ixz="0.0" iyy="${(1/12) * mass * ((body_length * body_length) + (body_height * body_height))}" iyz="0.0" izz="${(1/12) * mass * ((body_length * body_length) + (body_width  * body_width))}" />
         </inertial>
     </link>
-    <gazebo
-        reference="base_link">
+    <gazebo reference="base_link">
         <material>
             aluminum_frame
@@ -60,4 +53,10 @@
     </gazebo>
     <link name="base_footprint" />
+    <!-- <link name="odom" />
+    <joint name="odom_to_base_footprint_joint" type="fixed">
+        <origin xyz="0 0 0" rpy="0 0 0" />
+        <parent link="odom" />
+        <child link="base_footprint" />
+    </joint> -->
     <joint name="base_footprint_joint" type="fixed">
         <origin xyz="0 0 ${base_to_floor_z_offset}" rpy="0 0 0" />
@@ -69,19 +68,14 @@
     </xacro:wheel>
     <xacro:wheel wheel_prefix="front_right">
-        <origin xyz="0 -${(body_width/2)+wheel_center_offset} -${gear_box_center_height}"
-            rpy="0 0 0" />
+        <origin xyz="0 -${(body_width/2)+wheel_center_offset} -${gear_box_center_height}" rpy="0 0 0" />
     </xacro:wheel>
     <xacro:caster wheel_prefix="fcaster">
-        <origin xyz="${fwheel_offset} 0.0 -${wheel_radius + gear_box_center_height - caster_radius}"
-            rpy="0 0 0" />
+        <origin xyz="${fwheel_offset} 0.0 -${wheel_radius + gear_box_center_height - caster_radius}" rpy="0 0 0" />
     </xacro:caster>
     <xacro:caster wheel_prefix="rcaster">
-        <origin
-            xyz="${-fwheel_offset} 0.0 -${wheel_radius + gear_box_center_height - caster_radius}"
-            rpy="0 0 0" />
+        <origin xyz="${-fwheel_offset} 0.0 -${wheel_radius + gear_box_center_height - caster_radius}" rpy="0 0 0" />
     </xacro:caster>
     <xacro:ld06 lidar_prefix="right_rear">
-        <origin xyz="${-(body_length / 2) - 0.030}  -${((body_width / 2) - 0)} 0.200"
-            rpy="0 0 ${M_PI}" />
+        <origin xyz="${-(body_length / 2) - 0.030}  -${((body_width / 2) - 0)} 0.200" rpy="0 0 ${M_PI}" />
     </xacro:ld06>
     <xacro:ld06 lidar_prefix="left_front">
