Commit message: URDF changes for Raven

File: raven_description/urdf/raven.urdf.xacro (robot description, xacro)
@@ -7,32 +7,29 @@
     <xacro:property name="M_PI" value="3.14159" />
     <xacro:property name="body_height" value="0.262" />
-    <xacro:property name="body_length" value="0.6096" />
-    <xacro:property name="body_width" value="0.305" />
-    <xacro:property name="caster_radius" value="0.037" />
-    <xacro:property name="caster_width" value="0.030" />
-    <xacro:property name="d435_y_offset" value="0.077" />
-    <xacro:property name="fwheel_offset" value="-0.325" />
+    <xacro:property name="body_length" value="0.4572" />
+    <xacro:property name="body_width" value="0.3048" />
+    <xacro:property name="caster_radius" value="0.0381" />
+    <xacro:property name="caster_width" value="0.023" />
+    <xacro:property name="fwheel_offset" value="0.170" />
     <xacro:property name="gear_box_center_height" value="0.015" />
     <xacro:property name="ldlidar_height" value="0.035" />
     <xacro:property name="ldlidar_radius" value="0.034" />
-    <xacro:property name="ldlidar_left_front_x_offset" value="0.197" />
-    <xacro:property name="ldlidar_left_front_y_offset" value="0.193" />
-    <xacro:property name="ldlidar_left_front_z_offset" value="0.203" />
-    <xacro:property name="ldlidar_right_rear_x_offset" value="-0.400" />
-    <xacro:property name="ldlidar_right_rear_y_offset" value="-0.188" />
-    <xacro:property name="ldlidar_right_rear_z_offset" value="0.120" />
+    <xacro:property name="ldlidar_left_front_x_offset" value="0.26" />
+    <xacro:property name="ldlidar_left_front_y_offset" value="0.165" />
+    <xacro:property name="ldlidar_left_front_z_offset" value="0.067" />
+    <xacro:property name="ldlidar_right_rear_x_offset" value="-0.26" />
+    <xacro:property name="ldlidar_right_rear_y_offset" value="-0.165" />
+    <xacro:property name="ldlidar_right_rear_z_offset" value="0.228" />
     <xacro:property name="ldlidar_z_offset" value="-0.003" />
-    <xacro:property name="stereo_plate_x_offset" value="0.180" />
-    <xacro:property name="stereo_plate_z_offset" value="0.140" />
     <xacro:property name="t265_height" value="0.016" />
     <xacro:property name="t265_length" value="0.100" />
     <xacro:property name="t265_width" value="0.008" />
-    <xacro:property name="t265_x_offset" value="0.200" />
+    <xacro:property name="t265_x_offset" value="0.2126" />
     <xacro:property name="wheel_radius" value="0.10" />
     <xacro:property name="wheel_center_offset" value="0.030" />
     <xacro:property name="wheel_width" value="0.0254" />
     <xacro:property name="base_to_floor_z_offset" value="${wheel_radius+gear_box_center_height}" />
-    <xacro:property name="t265_z_offset" value="${base_to_floor_z_offset+0.175}" />
-    <xacro:property name="wheel_offset_from_front" value="0.190" />
+    <xacro:property name="t265_z_offset" value="${base_to_floor_z_offset+0.293}" />
+    <xacro:property name="wheel_offset_from_front" value="${body_length/2}" />
     <link name="base_link">
         <collision>
@@ -62,9 +59,9 @@
         <origin xyz="0 -${(body_width/2)+wheel_center_offset} -${gear_box_center_height}" rpy="0 0 0" />
     </xacro:wheel>
-    <xacro:caster wheel_prefix="lcaster">
-        <origin xyz="${fwheel_offset} 0.100 -0.078" rpy="0 0 0" />
+    <xacro:caster wheel_prefix="fcaster">
+        <origin xyz="${fwheel_offset} 0.0 -0.078" rpy="0 0 0" />
     </xacro:caster>
     <xacro:caster wheel_prefix="rcaster">
-        <origin xyz="${fwheel_offset} -0.080 -0.078" rpy="0 0 0" />
+        <origin xyz="${-fwheel_offset} -0.0 -0.078" rpy="0 0 0" />
     </xacro:caster>
     <!-- ldLidars-->
@@ -92,5 +89,5 @@
         <parent link="base_link" />
         <child link="lidar_frame_right_rear" />
-        <origin xyz="${ldlidar_right_rear_x_offset} ${ldlidar_right_rear_y_offset} ${ldlidar_right_rear_z_offset + ldlidar_height + ldlidar_z_offset}" rpy="0 0 ${M_PI/2.0}" />
+        <origin xyz="${ldlidar_right_rear_x_offset} ${ldlidar_right_rear_y_offset} ${ldlidar_right_rear_z_offset + ldlidar_height + ldlidar_z_offset}" rpy="0 0 ${M_PI}" />
     </joint>
     <link name="lidar_frame_left_front">
@@ -110,5 +107,5 @@
                 <cylinder length="${ldlidar_height}" radius="${ldlidar_radius}" />
             </geometry>
-            <origin rpy="0 0 0" xyz="0 0 0" />
+            <origin rpy="0 ${-(ldlidar_height + ldlidar_z_offset)} 0" xyz="0 0 0" />
             <material name="blackish" />
         </visual>
@@ -117,19 +114,6 @@
         <parent link="base_link" />
         <child link="lidar_frame_left_front" />
-        <origin xyz="${ldlidar_left_front_x_offset} ${ldlidar_left_front_y_offset} ${ldlidar_left_front_z_offset + ldlidar_height + ldlidar_z_offset}" rpy="0 0 ${-M_PI/2.0}" />
+        <origin xyz="${ldlidar_left_front_x_offset} ${ldlidar_left_front_y_offset} ${ldlidar_left_front_z_offset + ldlidar_height + ldlidar_z_offset}" rpy="0 0 ${0}" />
     </joint>
-    <!-- Stereo depth cameras-->
-    <xacro:include filename="$(find raven_description)/urdf/d435.urdf.xacro" />
-    <xacro:sensor_d435 parent="base_link" name="d435_left">
-        <origin xyz="${stereo_plate_x_offset} ${d435_y_offset} ${stereo_plate_z_offset}" rpy="0 0 0.35" />
-    </xacro:sensor_d435>
-    <xacro:sensor_d435 parent="base_link" name="d435_right">
-        <origin xyz="${stereo_plate_x_offset} ${-d435_y_offset} ${stereo_plate_z_offset}" rpy="0 0 -0.36" />
-    </xacro:sensor_d435>
-    <!-- <joint name="d435_left_to_base_footprint" type="fixed">
-        <parent link="d435_left" />
-        <child link="d435_left_link" />
-        <origin xyz="${stereo_plate_x_offset} ${d435_y_offset} ${stereo_plate_z_offset}" rpy="0 0 0.35" />
-    </joint> -->
     <!-- T265 y tilt is 31 degrees or 0.541 radians -->
     <!-- Visual odometry camera -->

File: raven_description/urdf/raven_gazebo.urdf.xacro (robot description, xacro)
@@ -171,5 +171,5 @@
     <material>Gazebo/Black</material>
   </gazebo>
-  <gazebo reference="lcaster_wheel_link">
+  <gazebo reference="fcaster_wheel_link">
     <mu1>0.00000</mu1>
     <mu2>0.00000</mu2>

File: raven_description/urdf/sonar.urdf.xacro (robot description, xacro)
@@ -26,5 +26,5 @@
     <xacro:property name="sonar_height" value="0.030" />
     <xacro:property name="sonar_width" value="0.050" />
-    <xacro:property name="sonar_z_offset" value="0.082" />
+    <xacro:property name="sonar_z_offset" value="0.173" />
     <link name="sonar_0">
         <visual>

File: raven_description/urdf/time_of_flight.urdf.xacro (robot description, xacro)
@@ -26,5 +26,5 @@
     <xacro:property name="tof_height" value="0.018" />
     <xacro:property name="tof_width" value="0.023" />
-    <xacro:property name="tof_z_offset" value="0.020" />
+    <xacro:property name="tof_z_offset" value="0.015" />
     <link name="tof_0">
         <visual>

Commit message: Humble fixes.

File: raven_description/urdf/raven.urdf.xacro (robot description, xacro)
@@ -5,4 +5,10 @@
     <xacro:include filename="$(find raven_description)/urdf/wheel.urdf.xacro" />
     <!-- <xacro:include filename="$(find raven_description)/urdf/raven_gazebo.urdf.xacro" /> -->
+    <material name="black">
+        <color rgba="0 0 0 1"/>
+    </material>
+    <material name="blackish">
+        <color rgba="0.1 0.1 0.1 1"/>
+    </material>
     <xacro:property name="M_PI" value="3.14159" />
     <xacro:property name="body_height" value="0.262" />
@@ -48,4 +54,16 @@
     </link>
     <link name="base_footprint" />
+    <link name="odom" />
+    <link name="odom_frame" />
+    <joint name="odom_to_odom_frame_joint" type="fixed">
+        <origin xyz="0 0 0" rpy="0 0 0" />>
+        <parent link="odom" />
+        <child link="odom_frame" />
+    </joint>
+    <joint name="odom_frame_to_t265_pose_frame_joint" type="fixed">
+        <origin xyz="0 0 0" rpy="0 0 0" />>
+        <parent link="odom_frame" />
+        <child link="t265_pose_frame" />
+    </joint>
     <joint name="base_footprint_joint" type="fixed">
         <origin xyz="0 0 ${base_to_floor_z_offset}" rpy="0 0 0" />

Commit message: Snapshot. World link still wrong.

File: raven_description/urdf/raven.urdf.xacro (robot description, xacro)
@@ -1,8 +1,26 @@
 <?xml version="1.0"?>
+<!--
+Copyright (c) 2023 Michael Wimble
+Permission is hereby granted, free of charge, to any person obtaining a copy
+of this software and associated documentation files (the "Software"), to deal
+in the Software without restriction, including without limitation the rights
+to use, copy, modify, merge, publish, distribute, sublicense, and/or sell
+copies of the Software, and to permit persons to whom the Software is
+furnished to do so, subject to the following conditions:
+The above copyright notice and this permission notice shall be included in all
+copies or substantial portions of the Software.
+THE SOFTWARE IS PROVIDED "AS IS", WITHOUT WARRANTY OF ANY KIND, EXPRESS OR
+IMPLIED, INCLUDING BUT NOT LIMITED TO THE WARRANTIES OF MERCHANTABILITY,
+FITNESS FOR A PARTICULAR PURPOSE AND NONINFRINGEMENT. IN NO EVENT SHALL THE
+AUTHORS OR COPYRIGHT HOLDERS BE LIABLE FOR ANY CLAIM, DAMAGES OR OTHER
+LIABILITY, WHETHER IN AN ACTION OF CONTRACT, TORT OR OTHERWISE, ARISING FROM,
+OUT OF OR IN CONNECTION WITH THE SOFTWARE OR THE USE OR OTHER DEALINGS IN THE
+SOFTWARE.
+-->
 <robot xmlns:xacro="http://ros.org/wiki/xacro" name="ravel">
     <xacro:include filename="$(find raven_description)/urdf/caster.urdf.xacro" />
     <xacro:include filename="$(find raven_description)/urdf/material.urdf.xacro" />
     <xacro:include filename="$(find raven_description)/urdf/wheel.urdf.xacro" />
-    <!-- <xacro:include filename="$(find raven_description)/urdf/raven_gazebo.urdf.xacro" /> -->
+    <xacro:include filename="$(find raven_description)/urdf/raven_gazebo.urdf.xacro" />
     <material name="black">
         <color rgba="0 0 0 1"/>
@@ -52,4 +70,9 @@
             <origin rpy="0 0 0" xyz="${(-body_length/2)+wheel_offset_from_front} 0 ${(body_height/2)}" />
         </visual>
+        <inertial>
+            <origin xyz="0 0 0.05" rpy="0 0 0"/>
+            <mass value="12" />
+            <inertia ixx="2.26" ixy="0.0" ixz="0.0" iyy="6.26" iyz="0.0" izz="8.5" />
+        </inertial>
     </link>
     <link name="base_footprint" />
@@ -140,5 +163,5 @@
             <geometry>
                 <box size="${t265_width} ${t265_length} ${t265_height}" />
-                <origin xyz="0 0 0" rpy="0.0 -0.0 0.0" />
+                <origin xyz="0 0 0" rpy="0.0 0.0 0.0" />
             </geometry>
         </collision>
@@ -147,5 +170,5 @@
                 <box size="${t265_width} ${t265_length} ${t265_height}" />
             </geometry>
-            <origin xyz="0 0 0" rpy="0.0 -0.0 0.0" />
+            <origin xyz="0 0 0" rpy="0.0 0.0 0.0" />
             <material name="t265_material" />
         </visual>
@@ -164,5 +187,5 @@
         <parent link="t265_pose_frame" />
         <child link="t265_rotate_frame" />
-        <origin xyz="0 0 0" rpy="0 0.541 0 " />
+        <origin xyz="0 0 0" rpy="0 0.541 0" />
     </joint>
     <xacro:include filename="$(find raven_description)/urdf/time_of_flight.urdf.xacro" />

File: raven_description/urdf/raven_gazebo.urdf.xacro (robot description, xacro)
@@ -6,8 +6,8 @@
       <material>Gazebo/Black</material>
     </gazebo>
-    <gazebo reference="${cam_name}_color_frame"/>
-    <gazebo reference="${cam_name}_color_optical_frame"/>
-    <gazebo reference="${cam_name}_depth_frame"/>
-    <gazebo reference="${cam_name}_depth_optical_frame"/>
+    <gazebo reference="${cam_name}_color_frame" />
+    <gazebo reference="${cam_name}_color_optical_frame" />
+    <gazebo reference="${cam_name}_depth_frame" />
+    <gazebo reference="${cam_name}_depth_optical_frame" />
     <gazebo reference="${cam_name}_joint" />
     <gazebo reference="${cam_name}_color_joint" />
@@ -17,45 +17,45 @@
     <!-- generate the RGB camera image -->
     <gazebo reference="cam_rgb_frame">
-        <sensor name="cam_rgb" type="camera">
-            <always_on>true</always_on>
-            <visualize>true</visualize>
-            <update_rate>15</update_rate>
-            <camera name="cam_rgb">
-                <horizontal_fov>1.085595</horizontal_fov>
-                <image>
-                    <width>1280</width>
-                    <height>960</height>
-                    <format>RGB8</format>
-                </image>
-                <clip>
-                    <near>0.03</near>
-                    <far>1000</far>
-                </clip>
-                <noise>
-                    <type>gaussian</type>
-                    <!-- Noise is sampled independently per pixel on each frame.
+      <sensor name="cam_rgb" type="camera">
+        <always_on>true</always_on>
+        <visualize>true</visualize>
+        <update_rate>15</update_rate>
+        <camera name="cam_rgb">
+          <horizontal_fov>1.085595</horizontal_fov>
+          <image>
+            <width>1280</width>
+            <height>960</height>
+            <format>RGB8</format>
+          </image>
+          <clip>
+            <near>0.03</near>
+            <far>1000</far>
+          </clip>
+          <noise>
+            <type>gaussian</type>
+            <!-- Noise is sampled independently per pixel on each frame.
                         That pixel's noise value is added to each of its color
                         channels, which at that point lie in the range [0,1]. -->
-                    <mean>0.0</mean>
-                    <stddev>0.007</stddev>
-                </noise>
-            </camera>
-            <plugin name="cam_rgb_driver" filename="libgazebo_ros_camera.so">
-                <ros>
-                <!-- <namespace></namespace> -->
-                    <!--
+            <mean>0.0</mean>
+            <stddev>0.007</stddev>
+          </noise>
+        </camera>
+        <plugin name="cam_rgb_driver" filename="libgazebo_ros_camera.so">
+          <ros>
+            <!-- <namespace></namespace> -->
+            <!--
                     <remapping>${cam_name}/image_raw:=cam_rgb/image_raw</remapping>
                     <remapping>${cam_name}/image_raw/compressed:=${cam_name}/color/image_raw/compressed</remapping>
                     <remapping>${cam_name}/image_raw/theora:=${cam_name}/color/image_raw/theora</remapping>
-                    <remapping>${cam_name}/image_raw/compressedDepth:=${cam_name}/color/image_raw/compressedDepth</remapping>
+            <remapping>${cam_name}/image_raw/compressedDepth:=${cam_name}/color/image_raw/compressedDepth</remapping>
                     <remapping>${cam_name}/camera_info:=${cam_name}/color/camera_info</remapping>
                     -->
-                </ros>
-                <!-- Set camera name. If empty, defaults to sensor name (i.e. "sensor_name") -->
-                <camera_name>cam_rgb</camera_name>
-                <!-- camera_name>omit so it defaults to sensor name</camera_name-->
-                <frame_name>cam_rgb_frame</frame_name>
-            </plugin>
-        </sensor>
+          </ros>
+          <!-- Set camera name. If empty, defaults to sensor name (i.e. "sensor_name") -->
+          <camera_name>cam_rgb</camera_name>
+          <!-- camera_name>omit so it defaults to sensor name</camera_name-->
+          <frame_name>cam_rgb_frame</frame_name>
+        </plugin>
+      </sensor>
     </gazebo>
     <!--  Add an RGBD camera -->
@@ -90,10 +90,13 @@
             <remapping>${cam_name}/image_raw/compressed:=${cam_name}/color/image_raw/compressed</remapping>
             <remapping>${cam_name}/image_raw/theora:=${cam_name}/color/image_raw/theora</remapping>
-            <remapping>${cam_name}/image_raw/compressedDepth:=${cam_name}/color/image_raw/compressedDepth</remapping>
+            <remapping>
+              ${cam_name}/image_raw/compressedDepth:=${cam_name}/color/image_raw/compressedDepth</remapping>
             <remapping>${cam_name}/camera_info:=${cam_name}/color/camera_info</remapping>
             <remapping>${cam_name}/depth/image_raw:=${cam_name}/depth/image_rect_raw</remapping>
-            <remapping>${cam_name}/depth/image_raw/compressed:=${cam_name}/depth/image_rect_raw/compressed</remapping>
+            <remapping>
+              ${cam_name}/depth/image_raw/compressed:=${cam_name}/depth/image_rect_raw/compressed</remapping>
             <remapping>${cam_name}/depth/image_raw/theora:=${cam_name}/depth/image_rect_raw/theora</remapping>
-            <remapping>${cam_name}/depth/image_raw/compressedDepth:=${cam_name}/depth/image_rect_raw/compressedDepth</remapping>
+            <remapping>
+              ${cam_name}/depth/image_raw/compressedDepth:=${cam_name}/depth/image_rect_raw/compressedDepth</remapping>
             <!-- remapping>${cam_name}/camera_info_depth:=${cam_name}/depth/camera_info</remapping -->
             <remapping>${cam_name}/points:=${cam_name}/depth/color/points</remapping>
@@ -108,9 +111,91 @@
     </gazebo>
   </xacro:macro>
-  <xacro:RealsenseGazebo cam_name="d435_left" />
-  <!--xacro:RealsenseGazebo cam_name="d435_right" /-->
+  <!-- This first link called "world" is empty -->
+  <link name="world"></link>
+  <!-- A simple fixed joint from our empty world link, to our base. -->
+  <!-- The base origin is offset from the world origin. -->
+  <joint name="base_joint" type="fixed">
+    <origin xyz="0 0 0" rpy="0 -0.541 0" />
+    <parent link="world" />
+    <child link="odom" />
+  </joint>
   <gazebo reference="base_link">
     <material>
-    Gazebo/DarkGrey
+      aluminum_frame
+    </material>
+  </gazebo>
+  <gazebo reference="lidar_frame_right_rear">
+    <material>
+      Gazebo/Black
+    </material>
+  </gazebo>
+  <gazebo reference="lidar_frame_left_front">
+    <material>
+      Gazebo/Black
+    </material>
+  </gazebo>
+  <gazebo reference="sonar_0">
+    <material>
+      Gazebo/Black
+    </material>
+  </gazebo>
+  <gazebo reference="sonar_1">
+    <material>
+      Gazebo/Black
+    </material>
+  </gazebo>
+  <gazebo reference="sonar_2">
+    <material>
+      Gazebo/Black
+    </material>
+  </gazebo>
+  <gazebo reference="sonar_3">
+    <material>
+      Gazebo/Black
+    </material>
+  </gazebo>
+  <gazebo reference="tof_0">
+    <material>
+      Gazebo/Grey
+    </material>
+  </gazebo>
+  <gazebo reference="tof_1">
+    <material>
+      Gazebo/Grey
+    </material>
+  </gazebo>
+  <gazebo reference="tof_2">
+    <material>
+      Gazebo/Grey
+    </material>
+  </gazebo>
+  <gazebo reference="tof_3">
+    <material>
+      Gazebo/Grey
+    </material>
+  </gazebo>
+  <gazebo reference="tof_4">
+    <material>
+      Gazebo/Grey
+    </material>
+  </gazebo>
+  <gazebo reference="tof_5">
+    <material>
+      Gazebo/Grey
+    </material>
+  </gazebo>
+  <gazebo reference="tof_6">
+    <material>
+      Gazebo/Grey
+    </material>
+  </gazebo>
+  <gazebo reference="tof_7">
+    <material>
+      Gazebo/Grey
+    </material>
+  </gazebo>
+  <gazebo reference="t265_pose_frame">
+    <material>
+      Gazebo/DarkGrey
     </material>
   </gazebo>
@@ -150,5 +235,5 @@
     </sensor>
     <material>
-    Gazebo/Black
+      Gazebo/Black
     </material>
   </gazebo>
@@ -179,40 +264,4 @@
     <min_depth>0.0001</min_depth>
     <material>Gazebo/Red</material>
-  </gazebo>
-  <gazebo reference="scan">
-    <!-- ray sensor -->
-    <sensor name="sensor_ray" type="ray">
-      <ray>
-        <scan>
-          <horizontal>
-            <samples>360</samples>
-            <resolution>1.0</resolution>
-            <min_angle>-1.369263</min_angle>
-            <max_angle>1.369263</max_angle>
-          </horizontal>
-        </scan>
-        <range>
-          <min>0.05</min>
-          <max>10.0</max>
-        </range>
-        <noise>
-          <type>gaussian</type>
-          <mean>0.0</mean>
-          <stddev>0.02</stddev>
-        </noise>
-      </ray>
-      <always_on>true</always_on>
-      <update_rate>15.0</update_rate>
-      <plugin name="laserscan" filename="libgazebo_ros_ray_sensor.so">
-        <ros>
-          <namespace>/simbot</namespace>
-          <remapping>~/out:=/scan_raw</remapping>
-        </ros>
-        <output_type>sensor_msgs/LaserScan</output_type>
-        <frame_name>scan</frame_name>
-      </plugin>
-      <visualize>1</visualize>
-    </sensor>
-    <material>Gazebo/Blue</material>
   </gazebo>
   <gazebo reference="rcaster_wheel_link">
@@ -236,5 +285,5 @@
       <right_joint>front_right_wheel</right_joint>
       <!-- kinematics -->
-      <wheel_separation>0.345</wheel_separation>
+      <wheel_separation>0.3108</wheel_separation>
       <wheel_diameter>0.2</wheel_diameter>
       <update_rate>100.0</update_rate>
@@ -249,5 +298,6 @@
       <robot_base_frame>base_footprint</robot_base_frame>
     </plugin>
-    <plugin name="gazebo_ros_joint_state_publisher" filename="libgazebo_ros_joint_state_publisher.so">
+    <plugin name="gazebo_ros_joint_state_publisher"
+      filename="libgazebo_ros_joint_state_publisher.so">
       <ros>
         <!-- Add a namespace -->
