Commit message: Simulation of the URDF is working. Robot does not move, however.

File: raven_description/urdf/raven.urdf.xacro (robot description, xacro)
@@ -20,7 +20,8 @@
 <robot xmlns:xacro="http://ros.org/wiki/xacro" name="ravel">
     <xacro:include filename="$(find raven_description)/urdf/caster.urdf.xacro" />
+    <xacro:include filename="$(find raven_description)/urdf/ld06.urdf.xacro" />
     <xacro:include filename="$(find raven_description)/urdf/material.urdf.xacro" />
+    <xacro:include filename="$(find raven_description)/urdf/raven_gazebo.urdf.xacro" />
     <xacro:include filename="$(find raven_description)/urdf/wheel.urdf.xacro" />
-    <xacro:include filename="$(find raven_description)/urdf/raven_gazebo.urdf.xacro" />
     <material name="black">
         <color rgba="0 0 0 1"/>
@@ -37,13 +38,4 @@
     <xacro:property name="fwheel_offset" value="0.170" />
     <xacro:property name="gear_box_center_height" value="0.015" />
-    <xacro:property name="ldlidar_height" value="0.035" />
-    <xacro:property name="ldlidar_radius" value="0.034" />
-    <xacro:property name="ldlidar_left_front_x_offset" value="0.26" />
-    <xacro:property name="ldlidar_left_front_y_offset" value="0.165" />
-    <xacro:property name="ldlidar_left_front_z_offset" value="0.067" />
-    <xacro:property name="ldlidar_right_rear_x_offset" value="-0.26" />
-    <xacro:property name="ldlidar_right_rear_y_offset" value="-0.165" />
-    <xacro:property name="ldlidar_right_rear_z_offset" value="0.228" />
-    <xacro:property name="ldlidar_z_offset" value="-0.003" />
     <xacro:property name="t265_height" value="0.016" />
     <xacro:property name="t265_length" value="0.100" />
@@ -70,9 +62,4 @@
             <origin rpy="0 0 0" xyz="${(-body_length/2)+wheel_offset_from_front} 0 ${(body_height/2)}" />
         </visual>
-        <inertial>
-            <origin xyz="0 0 0.05" rpy="0 0 0"/>
-            <mass value="12" />
-            <inertia ixx="2.26" ixy="0.0" ixz="0.0" iyy="6.26" iyz="0.0" izz="8.5" />
-        </inertial>
     </link>
     <link name="base_footprint" />
@@ -101,60 +88,15 @@
     </xacro:wheel>
     <xacro:caster wheel_prefix="fcaster">
-        <origin xyz="${fwheel_offset} 0.0 -0.078" rpy="0 0 0" />
+        <origin xyz="${fwheel_offset} 0.0 -${wheel_radius + gear_box_center_height - caster_radius}" rpy="0 0 0" />
     </xacro:caster>
     <xacro:caster wheel_prefix="rcaster">
-        <origin xyz="${-fwheel_offset} -0.0 -0.078" rpy="0 0 0" />
+        <origin xyz="${-fwheel_offset} 0.0 -${wheel_radius + gear_box_center_height - caster_radius}" rpy="0 0 0" />
     </xacro:caster>
-    <!-- ldLidars-->
-    <link name="lidar_frame_right_rear">
-        <collision>
-            <geometry>
-                <cylinder length="${ldlidar_height}" radius="${ldlidar_radius}" />
-            </geometry>
-            <origin rpy="0 0 0" xyz="0 0 0" />
-        </collision>
-        <inertial>
-            <origin xyz="0 0 0" rpy="0 0 0" />
-            <mass value="1" />
-            <inertia ixx="1.0" ixy="0.0" ixz="0.0" iyy="1.0" iyz="0.0" izz="1.0" />
-        </inertial>
-        <visual>
-            <geometry>
-                <cylinder length="${ldlidar_height}" radius="${ldlidar_radius}" />
-            </geometry>
-            <origin rpy="0 0 0" xyz="0 0 0" />
-            <material name="blackish" />
-        </visual>
-    </link>
-    <joint name="base_to_lidar_frame_right_rear" type="fixed">
-        <parent link="base_link" />
-        <child link="lidar_frame_right_rear" />
-        <origin xyz="${ldlidar_right_rear_x_offset} ${ldlidar_right_rear_y_offset} ${ldlidar_right_rear_z_offset + ldlidar_height + ldlidar_z_offset}" rpy="0 0 ${M_PI}" />
-    </joint>
-    <link name="lidar_frame_left_front">
-        <collision>
-            <geometry>
-                <cylinder length="${ldlidar_height}" radius="${ldlidar_radius}" />
-            </geometry>
-            <origin rpy="0 0 0" xyz="0 0 0" />
-        </collision>
-        <inertial>
-            <origin xyz="0 0 0" rpy="0 0 0" />
-            <mass value="1" />
-            <inertia ixx="1.0" ixy="0.0" ixz="0.0" iyy="1.0" iyz="0.0" izz="1.0" />
-        </inertial>
-        <visual>
-            <geometry>
-                <cylinder length="${ldlidar_height}" radius="${ldlidar_radius}" />
-            </geometry>
-            <origin rpy="0 ${-(ldlidar_height + ldlidar_z_offset)} 0" xyz="0 0 0" />
-            <material name="blackish" />
-        </visual>
-    </link>
-    <joint name="base_to_lidar_frame_left_front" type="fixed">
-        <parent link="base_link" />
-        <child link="lidar_frame_left_front" />
-        <origin xyz="${ldlidar_left_front_x_offset} ${ldlidar_left_front_y_offset} ${ldlidar_left_front_z_offset + ldlidar_height + ldlidar_z_offset}" rpy="0 0 ${0}" />
-    </joint>
+    <xacro:ld06 lidar_prefix="right_rear">
+        <origin xyz="${-(body_length / 2) - 0.030}  -${((body_width / 2) - 0)} 0.200" rpy="0 0 ${M_PI}"/>
+    </xacro:ld06>
+    <xacro:ld06 lidar_prefix="left_front">
+        <origin xyz="${(body_length / 2) + 0.030}  ${((body_width / 2) - 0.0)} 0.040" rpy="0 0 0"/>
+    </xacro:ld06>
     <!-- T265 y tilt is 31 degrees or 0.541 radians -->
     <!-- Visual odometry camera -->

File: raven_description/urdf/raven_gazebo.urdf.xacro (robot description, xacro)
@@ -112,100 +112,134 @@
   </xacro:macro>
   <!-- This first link called "world" is empty -->
-  <link name="world"></link>
+  <!-- <link name="world"></link> -->
   <!-- A simple fixed joint from our empty world link, to our base. -->
   <!-- The base origin is offset from the world origin. -->
-  <joint name="base_joint" type="fixed">
+  <!-- <joint name="base_joint" type="fixed">
     <origin xyz="0 0 0" rpy="0 -0.541 0" />
     <parent link="world" />
     <child link="odom" />
-  </joint>
+  </joint> -->
   <gazebo reference="base_link">
     <material>
       aluminum_frame
     </material>
+    <inertial>
+      <origin xyz="0 0 0.05" rpy="0 0 0" />
+      <mass value="12" />
+      <inertia ixx="2.26" ixy="0.0" ixz="0.0" iyy="6.26" iyz="0.0" izz="8.5" />
+    </inertial>
+  </gazebo>
+  <gazebo reference="ld06_base_cylinder_left_front">
+    <material>
+      Gazebo/Grey
+    </material>
+  </gazebo>
+  <gazebo reference="ld06_base_cylinder_right_rear">
+    <material>
+      Gazebo/Grey
+    </material>
+  </gazebo>
+  <gazebo reference="ld06_box_left_front">
+    <material>
+      Gazebo/Black
+    </material>
+  </gazebo>
+  <gazebo reference="ld06_box_right_rear">
+    <material>
+      Gazebo/Black
+    </material>
+  </gazebo>
+  <gazebo reference="ld06_cylinder_left_front">
+    <material>
+      Gazebo/BlueGlow
+    </material>
+  </gazebo>
+  <gazebo reference="ld06_cylinder_right_rear">
+    <material>
+      Gazebo/BlueGlow
+    </material>
+  </gazebo>
+  <gazebo reference="ld06_frame_left_front">
+    <material>
+      Gazebo/Grey
+    </material>
+  </gazebo>
+  <gazebo reference="ld06_frame_right_rear">
+    <material>
+      Gazebo/Grey
+    </material>
+  </gazebo>
+  <gazebo reference="sonar_0">
+    <material>
+      Gazebo/Black
+    </material>
+  </gazebo>
+  <gazebo reference="sonar_1">
+    <material>
+      Gazebo/Black
+    </material>
+  </gazebo>
+  <gazebo reference="sonar_2">
+    <material>
+      Gazebo/Black
+    </material>
+  </gazebo>
+  <gazebo reference="sonar_3">
+    <material>
+      Gazebo/Black
+    </material>
+  </gazebo>
+  <gazebo reference="tof_0">
+    <material>
+      Gazebo/Grey
+    </material>
+  </gazebo>
+  <gazebo reference="tof_1">
+    <material>
+      Gazebo/Grey
+    </material>
+  </gazebo>
+  <gazebo reference="tof_2">
+    <material>
+      Gazebo/Grey
+    </material>
+  </gazebo>
+  <gazebo reference="tof_3">
+    <material>
+      Gazebo/Grey
+    </material>
+  </gazebo>
+  <gazebo reference="tof_4">
+    <material>
+      Gazebo/Grey
+    </material>
+  </gazebo>
+  <gazebo reference="tof_5">
+    <material>
+      Gazebo/Grey
+    </material>
+  </gazebo>
+  <gazebo reference="tof_6">
+    <material>
+      Gazebo/Grey
+    </material>
+  </gazebo>
+  <gazebo reference="tof_7">
+    <material>
+      Gazebo/Grey
+    </material>
+  </gazebo>
+  <gazebo reference="t265_pose_frame">
+    <material>
+      Gazebo/DarkGrey
+    </material>
   </gazebo>
   <gazebo reference="lidar_frame_right_rear">
-    <material>
-      Gazebo/Black
-    </material>
-  </gazebo>
-  <gazebo reference="lidar_frame_left_front">
-    <material>
-      Gazebo/Black
-    </material>
-  </gazebo>
-  <gazebo reference="sonar_0">
-    <material>
-      Gazebo/Black
-    </material>
-  </gazebo>
-  <gazebo reference="sonar_1">
-    <material>
-      Gazebo/Black
-    </material>
-  </gazebo>
-  <gazebo reference="sonar_2">
-    <material>
-      Gazebo/Black
-    </material>
-  </gazebo>
-  <gazebo reference="sonar_3">
-    <material>
-      Gazebo/Black
-    </material>
-  </gazebo>
-  <gazebo reference="tof_0">
-    <material>
-      Gazebo/Grey
-    </material>
-  </gazebo>
-  <gazebo reference="tof_1">
-    <material>
-      Gazebo/Grey
-    </material>
-  </gazebo>
-  <gazebo reference="tof_2">
-    <material>
-      Gazebo/Grey
-    </material>
-  </gazebo>
-  <gazebo reference="tof_3">
-    <material>
-      Gazebo/Grey
-    </material>
-  </gazebo>
-  <gazebo reference="tof_4">
-    <material>
-      Gazebo/Grey
-    </material>
-  </gazebo>
-  <gazebo reference="tof_5">
-    <material>
-      Gazebo/Grey
-    </material>
-  </gazebo>
-  <gazebo reference="tof_6">
-    <material>
-      Gazebo/Grey
-    </material>
-  </gazebo>
-  <gazebo reference="tof_7">
-    <material>
-      Gazebo/Grey
-    </material>
-  </gazebo>
-  <gazebo reference="t265_pose_frame">
-    <material>
-      Gazebo/DarkGrey
-    </material>
-  </gazebo>
-  <gazebo reference="scan">
-    <!-- ray sensor -->
-    <sensor name="sensor_ray" type="ray">
+    <sensor name="sensor_ray_right" type="ray">
       <ray>
         <scan>
           <horizontal>
-            <samples>360</samples>
-            <resolution>1.0</resolution>
+            <samples>450</samples>
+            <resolution>0.8</resolution>
             <min_angle>0</min_angle>
             <max_angle>6.28</max_angle>
@@ -224,8 +258,43 @@
       <always_on>true</always_on>
       <update_rate>3.0</update_rate>
-      <plugin name="laserscan" filename="libgazebo_ros_ray_sensor.so">
+      <plugin name="laserscan_right" filename="libgazebo_ros_ray_sensor.so">
         <ros>
-          <!-- <namespace>/</namespace> -->
-          <remapping>~/out:=/scan</remapping>
+          <remapping>~/out:=/scan_right</remapping>
+        </ros>
+        <output_type>sensor_msgs/LaserScan</output_type>
+        <frame_name>scan</frame_name>
+      </plugin>
+      <visualize>1</visualize>
+    </sensor>
+    <material>
+      Gazebo/Black
+    </material>
+  </gazebo>
+  <gazebo reference="lidar_frame_left_front">
+    <sensor name="sensor_ray_left" type="ray">
+      <ray>
+        <scan>
+          <horizontal>
+            <samples>450</samples>
+            <resolution>0.8</resolution>
+            <min_angle>0</min_angle>
+            <max_angle>6.28</max_angle>
+          </horizontal>
+        </scan>
+        <range>
+          <min>0.05</min>
+          <max>10.0</max>
+        </range>
+        <noise>
+          <type>gaussian</type>
+          <mean>0.0</mean>
+          <stddev>0.02</stddev>
+        </noise>
+      </ray>
+      <always_on>true</always_on>
+      <update_rate>3.0</update_rate>
+      <plugin name="laserscan_left" filename="libgazebo_ros_ray_sensor.so">
+        <ros>
+          <remapping>~/out:=/scan_right</remapping>
         </ros>
         <output_type>sensor_msgs/LaserScan</output_type>

File: raven_description/urdf/time_of_flight.urdf.xacro (robot description, xacro)
@@ -39,5 +39,5 @@
         <child link="tof_0" />
         <parent link="base_link" />
-        <origin xyz="${front_edge+(tof_depth/2)} ${case_left_edge-(tof_width/2)} ${(tof_height/2)+tof_z_offset}" rpy="0 0 0" />
+        <origin xyz="${front_edge+(tof_depth/2)} ${case_left_edge-(tof_width/2) - 0.020} ${(tof_height/2)+tof_z_offset}" rpy="0 0 0" />
     </joint>
     <link name="tof_1">
@@ -53,5 +53,5 @@
         <child link="tof_1" />
         <parent link="base_link" />
-        <origin xyz="${front_edge+(tof_depth/2)} ${case_right_edge+(tof_width/2)} ${(tof_height/2)+tof_z_offset}" rpy="0 0 0" />
+        <origin xyz="${front_edge+(tof_depth/2)} ${case_right_edge +(tof_width/2) + 0.020} ${(tof_height/2)+tof_z_offset}" rpy="0 0 0" />
     </joint>
     <link name="tof_2">
@@ -67,5 +67,5 @@
         <child link="tof_2" />
         <parent link="base_link" />
-        <origin xyz="${front_edge-(tof_width/2)} ${case_left_edge+(tof_depth/2)} ${(tof_height/2)+tof_z_offset}" rpy="0 0 ${M_PI / 2}" />
+        <origin xyz="${front_edge-(tof_width/2 + 0.020)} ${case_left_edge+(tof_depth/2)} ${(tof_height/2)+tof_z_offset}" rpy="0 0 ${M_PI / 2}" />
     </joint>
     <link name="tof_3">
@@ -81,5 +81,5 @@
         <child link="tof_3" />
         <parent link="base_link" />
-        <origin xyz="${front_edge-(tof_width/2)} ${case_right_edge-(tof_depth/2)} ${(tof_height/2)+tof_z_offset}" rpy="0 0 -${M_PI / 2}" />
+        <origin xyz="${front_edge-(tof_width/2 + 0.020)} ${case_right_edge-(tof_depth/2)} ${(tof_height/2)+tof_z_offset}" rpy="0 0 -${M_PI / 2}" />
     </joint>
     <link name="tof_4">
@@ -95,5 +95,5 @@
         <child link="tof_4" />
         <parent link="base_link" />
-        <origin xyz="${back_edge+(tof_width/2)} ${case_left_edge+(tof_depth/2)} ${(tof_height/2)+tof_z_offset}" rpy="0 0 ${M_PI / 2}" />
+        <origin xyz="${back_edge+(tof_width/2) + 0.020} ${case_left_edge+(tof_depth/2)} ${(tof_height/2)+tof_z_offset}" rpy="0 0 ${M_PI / 2}" />
     </joint>
     <link name="tof_5">
@@ -109,5 +109,5 @@
         <child link="tof_5" />
         <parent link="base_link" />
-        <origin xyz="${back_edge+(tof_width/2)} ${case_right_edge-(tof_depth/2)} ${(tof_height/2)+tof_z_offset}" rpy="0 0 -${M_PI / 2}" />
+        <origin xyz="${back_edge+(tof_width/2) + 0.020} ${case_right_edge-(tof_depth/2)} ${(tof_height/2)+tof_z_offset}" rpy="0 0 -${M_PI / 2}" />
     </joint>
     <link name="tof_6">
@@ -123,5 +123,5 @@
         <child link="tof_6" />
         <parent link="base_link" />
-        <origin xyz="${back_edge-(tof_depth/2)} ${case_left_edge-(tof_width/2)} ${(tof_height/2)+tof_z_offset}" rpy="0 0 -${M_PI}" />
+        <origin xyz="${back_edge-(tof_depth/2)} ${case_left_edge-(tof_width/2) - 0.020} ${(tof_height/2)+tof_z_offset}" rpy="0 0 -${M_PI}" />
     </joint>
     <link name="tof_7">
@@ -137,5 +137,5 @@
         <child link="tof_7" />
         <parent link="base_link" />
-        <origin xyz="${back_edge-(tof_depth/2)} ${case_right_edge+(tof_width/2)} ${(tof_height/2)+tof_z_offset}" rpy="0 0 -${M_PI}" />
+        <origin xyz="${back_edge-(tof_depth/2)} ${case_right_edge+(tof_width/2) + 0.020} ${(tof_height/2)+tof_z_offset}" rpy="0 0 -${M_PI}" />
     </joint>
 </robot>

Commit message: New sim launch. Added oak-d cameras to URDF

File: raven_description/urdf/raven.urdf.xacro (robot description, xacro)
@@ -25,4 +25,5 @@
     <xacro:include filename="$(find raven_description)/urdf/raven_gazebo.urdf.xacro" />
     <xacro:include filename="$(find raven_description)/urdf/wheel.urdf.xacro" />
+    <xacro:include filename="$(find raven_description)/urdf/oakd.urdf.xacro" />
     <link name="base_link">
         <collision>
@@ -136,3 +137,11 @@
     <xacro:include filename="$(find raven_description)/urdf/time_of_flight.urdf.xacro" />
     <xacro:include filename="$(find raven_description)/urdf/sonar.urdf.xacro" />
+    <xacro:oakd_link mount_point="right" />
+    <xacro:oakd_joint mount_point="right">
+        <origin xyz="0.170 -0.055 0.350" rpy="0 0 -0.523599" />
+    </xacro:oakd_joint>
+    <xacro:oakd_link mount_point="left" />
+    <xacro:oakd_joint mount_point="left">
+        <origin xyz="0.170 0.055 0.350" rpy="0 0 0.523599" />
+    </xacro:oakd_joint>
 </robot>

Commit message: Oakd left camera emitting depth images

File: raven_description/urdf/raven.urdf.xacro (robot description, xacro)
@@ -21,4 +21,6 @@
     <xacro:include filename="$(find raven_description)/urdf/raven_properties.urdf.xacro" />
     <xacro:include filename="$(find raven_description)/urdf/caster.urdf.xacro" />
+    <xacro:include filename="$(find raven_description)/urdf/depthai_macro.urdf.xacro" />
+    <xacro:include filename="$(find raven_description)/urdf/inertials.xacro" />
     <xacro:include filename="$(find raven_description)/urdf/ld06.urdf.xacro" />
     <xacro:include filename="$(find raven_description)/urdf/material.urdf.xacro" />
@@ -137,11 +139,47 @@
     <xacro:include filename="$(find raven_description)/urdf/time_of_flight.urdf.xacro" />
     <xacro:include filename="$(find raven_description)/urdf/sonar.urdf.xacro" />
-    <xacro:oakd_link mount_point="right" />
+    <xacro:depthai_camera
+        camera_name="oakd_left"
+        camera_model="OAK-D"
+        parent="base_link"
+        base_frame="oakd_left_base_link"
+        cam_pos_x="0.170"
+        cam_pos_y="0.055"
+        cam_pos_z="0.350"
+        cam_roll="0.0"
+        cam_pitch="0.0"
+        cam_yaw="0.523599"
+    />
+    <xacro:depthai_camera
+        camera_name="oakd_right"
+        camera_model="OAK-D"
+        parent="base_link"
+        base_frame="oakd_right_base_link"
+        cam_pos_x="0.170"
+        cam_pos_y="-0.055"
+        cam_pos_z="0.350"
+        cam_roll="0.0"
+        cam_pitch="0.0"
+        cam_yaw="-0.523599"
+    />
+    <!-- <xacro:oakd_link mount_point="right" />
     <xacro:oakd_joint mount_point="right">
         <origin xyz="0.170 -0.055 0.350" rpy="0 0 -0.523599" />
     </xacro:oakd_joint>
+    <link name="oakd_left_right_camera_optical_frame" />
+    <joint name="oakd_left_link_optical_frame" type="fixed">
+        <parent link="oakd_left"/>
+        <child link="oakd_left_right_camera_optical_frame"/>
+        <origin xyz="0 0 0" rpy="0 0 0" />
+    </joint>
     <xacro:oakd_link mount_point="left" />
     <xacro:oakd_joint mount_point="left">
         <origin xyz="0.170 0.055 0.350" rpy="0 0 0.523599" />
     </xacro:oakd_joint>
+    <link name="oakd_right_right_camera_optical_frame" />
+    <joint name="oakd_right_link_optical_frame" type="fixed">
+        <parent link="oakd_right"/>
+        <child link="oakd_right_right_camera_optical_frame"/>
+        <origin xyz="0 0 0" rpy="0 0 0" />
+    </joint> -->
 </robot>

Commit message: Big shift

File: raven_description/urdf/raven.urdf.xacro (robot description, xacro)
@@ -61,15 +61,14 @@
     </gazebo>
     <link name="base_footprint" />
-    <link name="odom" />
-    <link name="odom_frame" />
-    <joint name="odom_to_odom_frame_joint" type="fixed">
-        <origin xyz="0 0 0" rpy="0 0 0" />> <parent link="odom" />
+    <!--joint name="odom_to_odom_frame_joint" type="fixed">
+        <origin xyz="0 0 0" rpy="0 0 0" />
+        <parent link="odom" />
         <child link="odom_frame" />
-    </joint>
-    <joint name="odom_frame_to_t265_pose_frame_joint" type="fixed">
+    </joint> -->
+    <!-- joint name="odom_frame_to_t265_pose_frame_joint" type="fixed">
         <origin xyz="0 0 0" rpy="0 0 0" />> <parent link="odom_frame" />
         <child
             link="t265_pose_frame" />
-    </joint>
+    </joint> -->
     <joint name="base_footprint_joint" type="fixed">
         <origin xyz="0 0 ${base_to_floor_z_offset}" rpy="0 0 0" />
@@ -102,5 +101,5 @@
     <!-- T265 y tilt is 31 degrees or 0.541 radians -->
     <!-- Visual odometry camera -->
-    <link name="t265_pose_frame">
+    <!-- <link name="t265_pose_frame">
         <collision>
             <geometry>
@@ -126,8 +125,4 @@
         <child link="base_footprint" />
         <origin xyz="-${t265_x_offset} 0 -${t265_z_offset}" rpy="0 0 0" />
-        <!--
-        <child link="base_footprint" />
-        <origin xyz="-${t265_x_offset} 0 -${t265_z_offset}" rpy="0 0.541 0 " />
-        -->
     </joint>
     <link name="t265_rotate_frame" />
@@ -135,9 +130,9 @@
         <parent link="t265_pose_frame" />
         <child link="t265_rotate_frame" />
-        <origin xyz="0 0 0" rpy="0 0.541 0" />
-    </joint>
+        <origin xyz="0 0 0" rpy="0 0 0" />
+    </joint> -->
     <xacro:include filename="$(find raven_description)/urdf/time_of_flight.urdf.xacro" />
     <xacro:include filename="$(find raven_description)/urdf/sonar.urdf.xacro" />
-    <xacro:depthai_camera
+    <!-- <xacro:depthai_camera
         camera_name="oakd_left"
         camera_model="OAK-D"
@@ -162,5 +157,5 @@
         cam_pitch="0.0"
         cam_yaw="-0.523599"
-    />
+    /> -->
     <!-- <xacro:oakd_link mount_point="right" />
     <xacro:oakd_joint mount_point="right">
